Commit message: float apriltags and high watchtower's camera

File: catkin_ws/src/duckiepond_vehicle/urdf/apriltag.xacro (robot description, xacro)
@@ -4,5 +4,5 @@
   <!-- Defines the base vehicle -->
   <xacro:include filename="$(find duckiepond_vehicle)/urdf/apriltag_base.xacro" />
-  <xacro:apriltag_base name="$(arg robot_name)_apriltag_base_plugin" tag_id="$(arg tag_id)" tag_id2="$(arg tag_id2)" tag_size="$(arg tag_size)"/>
+  <xacro:apriltag_base name="$(arg robot_name)_apriltag_base_plugin" tag_id="$(arg tag_id)" tag_size="$(arg tag_size)"/>
   <!-- Attach hydrodynamics plugin -->
   <xacro:include filename="$(find duckiepond_vehicle)/urdf/usv_gazebo_dynamics_plugin.xacro" />

File: catkin_ws/src/duckiepond_vehicle/urdf/apriltag_base.xacro (robot description, xacro)
@@ -1,11 +1,6 @@
 <?xml version="1.0"?>
 <robot xmlns:xacro="http://ros.org/wiki/xacro">
-  <xacro:macro name="apriltag_base" params=" name tag_id:=0 tag_id2:=0 tag_size:=0.8">
+  <xacro:macro name="apriltag_base" params=" name tag_id:=0 tag_size:=0.8">
   <xacro:property name="size" value="${tag_size}"/>
-<!--
-  <xacro:property name="tag_size" value="0.7" />
-  <xacro:property name="M_PI" value="3.1415926535897931" />
-  <xacro:property name="tag_1" value="0" />
--->
   <!-- totem -->
   <link name="base_link">
@@ -37,61 +32,6 @@
   <!-- apriltag_1 -->
   <link name="apriltag_1">
-    <collision>
-      <origin xyz="-0.25 -0.25 0.75" rpy="0 0 0"/>
-      <geometry>
-        <box size="0.01 ${size} ${size}"/>
-      </geometry>
-    </collision>
     <visual>
-      <origin xyz="-0.25 -0.25 0.75" rpy="0 0 0"/>
-      <geometry>
-        <box size="0.01 ${size} ${size}"/>
-      </geometry>
-    </visual>
-    <inertial>
-      <origin xyz="-0.25 -0.25 0.75" rpy="0 0 0"/>
-      <mass value="1"/>
-      <inertia
-        ixx="1.0" ixy="0.0" ixz="0.0"
-        iyy="1.0" iyz="0.0"
-        izz="1.0"/>
-    </inertial>
-  </link>
-  <!-- apriltag_1_back -->
-  <link name="apriltag_1_back">
-    <visual>
-      <origin xyz="-0.24 -0.25 0.75" rpy="0 0 0"/>
-      <geometry>
-        <box size="0.01 ${size} ${size}"/>
-      </geometry>
-    </visual>
-  </link>
-  <!-- apriltag_2 -->
-  <link name="apriltag_2">
-    <collision>
-      <origin xyz="0.25 0.25  0.75" rpy="0 0 1.57"/>
-      <geometry>
-        <box size="0.01 ${size} ${size}"/>
-      </geometry>
-    </collision>
-    <visual>
-      <origin xyz="0.25 0.25  0.75" rpy="0 0 1.57"/>
-      <geometry>
-        <box size="0.01 ${size} ${size}"/>
-      </geometry>
-    </visual>
-    <inertial>
-      <origin xyz="0.25 0.25  0.75" rpy="0 0 1.57"/>
-      <mass value="1"/>
-      <inertia
-        ixx="1.0" ixy="0.0" ixz="0.0"
-        iyy="1.0" iyz="0.0"
-        izz="1.0"/>
-    </inertial>
-  </link>
-  <!-- apriltag_2_back -->
-  <link name="apriltag_2_back">
-    <visual>
-      <origin xyz="0.25 0.24  0.75" rpy="0 0 1.57"/>
+      <origin xyz="0.25 -0.25 0.25" rpy="0 1.57 0"/>
       <geometry>
         <box size="0.01 ${size} ${size}"/>
@@ -104,22 +44,6 @@
     <child link="apriltag_1"/>
   </joint>
-  <joint name="totem_to_apriltag_1_back" type="fixed">
-    <parent link="base_link"/>
-    <child link="apriltag_1_back"/>
-  </joint>
-  <joint name="totem_to_apriltag_2" type="fixed">
-    <parent link="base_link"/>
-    <child link="apriltag_2"/>
-  </joint>
-  <joint name="totem_to_apriltag_2_back" type="fixed">
-    <parent link="base_link"/>
-    <child link="apriltag_2_back"/>
-  </joint>
   <!-- apriltage id -->
   <gazebo reference="apriltag_1">
-    <turnGravityOff>false</turnGravityOff>
-    <material>a_${tag_id2}/Image</material>
-  </gazebo>
-  <gazebo reference="apriltag_2">
     <turnGravityOff>false</turnGravityOff>
     <material>a_${tag_id}/Image</material>

File: catkin_ws/src/duckiepond_vehicle/urdf/duckieboat.xacro (robot description, xacro)
@@ -27,5 +27,5 @@
     <!-- Attach apriltag -->
     <xacro:include filename="$(find duckiepond_vehicle)/urdf/usv_gazebo_apriltags_plugin.xacro" />
-    <xacro:usv_apriltags name="top_tag" tag_id="512" tag_size="1.00">
+    <xacro:usv_apriltags name="top_tag" tag_id="$(arg robot_id)" tag_size="1.00">
         <origin xyz="0.5 0 1" rpy="0 1.57 0"/>
     </xacro:usv_apriltags>

File: catkin_ws/src/duckiepond_vehicle/urdf/usv_gazebo_camera_plugin.xacro (robot description, xacro)
@@ -1,13 +1,13 @@
 <?xml version="1.0"?>
 <robot xmlns:xacro="http://ros.org/wiki/xacro">
-  <xacro:macro name="usv_camera" params="name robot_name:=duckieboat camera_z:=0.45 camera_row:=1.57">
+  <xacro:macro name="usv_camera" params="name robot_name:=duckieboat camera_z:=0.45 camera_pitch:=0">
   <!-- camera position -->
   <xacro:property name="origin_mid">
-    <origin xyz="1 0 ${camera_z}" rpy="0 0 0" />
+    <origin xyz="1 0 ${camera_z}" rpy="0 ${camera_pitch} 0" />
   </xacro:property>
   <!-- mid camera -->
   <link name="camera_link">
     <visual>
-      <origin xyz="-0.01 0 0" rpy="${camera_row} 0 1.57"/>
+      <origin xyz="-0.01 0 0" rpy="0 ${camera_pitch} 1.57"/>
       <geometry>
         <mesh filename="model://zed/zed_model.dae" scale="0.02 0.02 0.02"/>

File: catkin_ws/src/duckiepond_vehicle/urdf/watchtower.xacro (robot description, xacro)
@@ -24,4 +24,4 @@
     <!-- Attach camera plugin -->
     <xacro:include filename="$(find duckiepond_vehicle)/urdf/usv_gazebo_camera_plugin.xacro"/>
-    <xacro:usv_camera name="camera" robot_name="$(arg robot_name)" camera_z="$(arg camera_z)" camera_row="$(arg camera_row)"/>
+    <xacro:usv_camera name="camera" robot_name="$(arg robot_name)" camera_z="$(arg camera_z)" camera_pitch="$(arg camera_pitch)"/>
 </robot>
