Commit message: add boat name on all sensor topic name

File: catkin_ws/src/duckiepond_vehicle/urdf/duckieboat.xacro (robot description, xacro)
@@ -1,23 +1,24 @@
 <?xml version="1.0"?>
-<robot xmlns:xacro="http://ros.org/wiki/xacro"
-       name="duckieboat">
-  <!-- Defines the base vehicle -->
-  <xacro:include filename="$(find duckiepond_vehicle)/urdf/duckieboat_base.xacro" />
-  <!-- Attach front camera plugin -->
-  <xacro:include filename="$(find duckiepond_vehicle)/urdf/duckieboat_gazebo_camera_plugin.xacro" />
-  <xacro:duckieboat_camera name="$(arg name)_front_camera" robot_name="$(arg name)"/>
-  <!-- Attach GPS plugin -->
-  <xacro:include filename="$(find duckiepond_vehicle)/urdf/duckieboat_gazebo_gps_plugin.xacro" />
-  <xacro:wamv_gps name="$(arg name)_gps" latitude="24.788808" longitude="121.000188" altitude="2.5">
-    <origin xyz="0.2 0.0 2.5" rpy="0 0 0" />
-  </xacro:wamv_gps>
-  <!-- Attach hydrodynamics plugin -->
-  <xacro:include filename="$(find duckiepond_vehicle)/urdf/usv_gazebo_dynamics_plugin.xacro" />
-  <xacro:usv_dynamics_gazebo name="$(arg name)_dynamics_plugin"/>
-  <!-- Attach thrust plugin -->
-  <xacro:include filename="$(find duckiepond_vehicle)/urdf/usv_gazebo_thrust_plugin.xacro" />
-  <xacro:usv_thrust_gazebo name="$(arg name)_thrust_plugin"/>
-  <!-- Attach p3d odometry plugin -->
-  <xacro:include filename="$(find duckiepond_vehicle)/urdf/usv_gazebo_p3d_plugin.xacro" />
-  <xacro:usv_p3d name="$(arg name)_p3d"/>
+<robot xmlns:xacro="http://ros.org/wiki/xacro" name="duckieboat">
+    <!-- Defines the base vehicle -->
+    <xacro:include filename="$(find duckiepond_vehicle)/urdf/duckieboat_base.xacro" />
+    <!-- Attach IMU plugin -->
+    <xacro:include filename="$(find duckiepond_vehicle)/urdf/usv_gazebo_imu_plugin.xacro" />
+    <xacro:usv_imu name="imu" robot_name="$(arg robot_name)">
+        <origin xyz="0.2 0.0 0.5" rpy="0 0 0" />
+    </xacro:usv_imu>
+    <!-- Attach p3d odometry plugin -->
+    <xacro:include filename="$(find duckiepond_vehicle)/urdf/usv_gazebo_p3d_plugin.xacro" />
+    <xacro:usv_p3d name="p3d" robot_name="$(arg robot_name)"/>
+    <!-- Attach GPS plugin -->
+    <xacro:include filename="$(find duckiepond_vehicle)/urdf/usv_gazebo_gps_plugin.xacro" />
+    <xacro:usv_gps name="gps" latitude="24.788808" longitude="121.000188" altitude="2.5" robot_name="$(arg robot_name)">
+        <origin xyz="0.2 0.0 0.8" rpy="0 0 0" />
+    </xacro:usv_gps>
+    <!-- Attach hydrodynamics plugin -->
+    <xacro:include filename="$(find duckiepond_vehicle)/urdf/usv_gazebo_dynamics_plugin.xacro" robot_name="$(arg robot_name)"/>
+    <xacro:usv_dynamics_gazebo name="dynamics" robot_name="$(arg robot_name)"/>
+    <!-- Attach thrust plugin -->
+    <xacro:include filename="$(find duckiepond_vehicle)/urdf/usv_gazebo_thrust_plugin.xacro" robot_name="$(arg robot_name)"/>
+    <xacro:usv_thrust_gazebo name="thrust" robot_name="$(arg robot_name)"/>
 </robot>

File: catkin_ws/src/duckiepond_vehicle/urdf/duckieboat_base.xacro (robot description, xacro)
@@ -27,5 +27,5 @@
       <geometry>
         <mesh scale="0.001 0.001 0.001"
-          filename="package://wamv_description/mesh/DUCKIEBOAT-Base.stl" />
+          filename="package://duckiepond_vehicle/mesh/DUCKIEBOAT-Base.stl" />
       </geometry>
     </visual>
@@ -36,5 +36,5 @@
       <geometry>
         <mesh scale="0.001 0.001 0.001"
-          filename="package://wamv_description/mesh/DUCKIEBOAT-Base.stl" />
+          filename="package://duckiepond_vehicle/mesh/DUCKIEBOAT-Base.stl" />
       </geometry>
     </collision>
@@ -44,10 +44,10 @@
     <visual>
      <geometry>
-       <mesh filename="package://wamv_description/mesh/PROPELLER.dae"/>
+       <mesh filename="package://duckiepond_vehicle/mesh/PROPELLER.dae"/>
      </geometry>
     </visual>
     <collision name="right_motor_collision">
       <geometry>
-        <mesh filename="package://wamv_description/mesh/PROPELLER.dae"/>
+        <mesh filename="package://duckiepond_vehicle/mesh/PROPELLER.dae"/>
       </geometry>
     </collision>
@@ -77,10 +77,10 @@
     <visual>
      <geometry>
-       <mesh filename="package://wamv_description/mesh/PROPELLER.dae"/>
+       <mesh filename="package://duckiepond_vehicle/mesh/PROPELLER.dae"/>
      </geometry>
     </visual>
     <collision name="left_motor_collision">
       <geometry>
-        <mesh filename="package://wamv_description/mesh/PROPELLER.dae"/>
+        <mesh filename="package://duckiepond_vehicle/mesh/PROPELLER.dae"/>
       </geometry>
     </collision>

File: catkin_ws/src/duckiepond_vehicle/urdf/usv_gazebo_camera_plugin.xacro (robot description, xacro)
@@ -1,5 +1,5 @@
 <?xml version="1.0"?>
 <robot xmlns:xacro="http://ros.org/wiki/xacro">
-  <xacro:macro name="duckieboat_camera" params="name robot_name:=/ ">
+  <xacro:macro name="usv_camera" params="name robot_name:=duckieboat">
   <!-- camera position -->
   <xacro:property name="origin_mid">
@@ -44,5 +44,5 @@
         </noise>
       </camera>
-      <plugin name="camera_controller" filename="libgazebo_ros_camera.so">
+      <plugin name="${name}_camera_controller" filename="libgazebo_ros_camera.so">
         <alwaysOn>true</alwaysOn>
         <updateRate>0.0</updateRate>

File: catkin_ws/src/duckiepond_vehicle/urdf/usv_gazebo_dynamics_plugin.xacro (robot description, xacro)
@@ -1,8 +1,8 @@
 <?xml version="1.0"?>
 <robot xmlns:xacro="http://ros.org/wiki/xacro">
-  <xacro:macro name="usv_dynamics_gazebo" params="name">
+  <xacro:macro name="usv_dynamics_gazebo" params="name robot_name:=boat">
     <!--Gazebo Plugin for simulating WAM-V dynamics-->
     <gazebo >
-      <plugin name="usv_dynamics_${name}" filename="libusv_gazebo_dynamics_plugin.so">
+      <plugin name="usv_dynamics_${robot_name}" filename="libusv_gazebo_dynamics_plugin.so">
 	<bodyName>base_link</bodyName>
 	<waterLevel>0</waterLevel> <!-- Must be same as the ocean model!-->

File: catkin_ws/src/duckiepond_vehicle/urdf/usv_gazebo_gps_plugin.xacro (robot description, xacro)
@@ -1,9 +1,9 @@
 <?xml version="1.0"?>
 <robot xmlns:xacro="http://ros.org/wiki/xacro">
-  <xacro:macro name="wamv_gps" params="*origin name longitude:=-157.8901 latitude:=21.30996 altitude:=1.5">
+  <xacro:macro name="usv_gps" params="*origin name longitude:=-157.8901 latitude:=21.30996 altitude:=1.5 robot_name:=boat">
     <link name="${name}">
       <visual>
         <geometry>
-          <box size="0.2 1.4 0.2" />
+          <box size="0.2 0.5 0.2" />
         </geometry>
       </visual>
@@ -15,10 +15,10 @@
     </joint>
     <gazebo>
-      <plugin name="gps_plugin_${name}" filename="libhector_gazebo_ros_gps.so">
+      <plugin name="gps_plugin_${robot_name}" filename="libhector_gazebo_ros_gps.so">
 		<updateRate>5.0</updateRate>
 		<alwaysOn>true</alwaysOn>
 	        <bodyName>base_link</bodyName>
 	        <frameId>gps</frameId>
-		<topicName>gps</topicName>
+		<topicName>${robot_name}/gps</topicName>
     	<velocityTopicName>fix_velocity</velocityTopicName>
 		<!-- Location of origin of Gazebo Sand Island map -->

File: catkin_ws/src/duckiepond_vehicle/urdf/usv_gazebo_p3d_plugin.xacro (robot description, xacro)
@@ -1,11 +1,11 @@
 <?xml version="1.0"?>
 <robot xmlns:xacro="http://ros.org/wiki/xacro">
-  <xacro:macro name="usv_p3d" params="name">
+  <xacro:macro name="usv_p3d" params="name robot_name:=boat">
     <gazebo>
-      <plugin name="usv_p3d_${name}" filename="libgazebo_ros_p3d.so">
+      <plugin name="usv_p3d_${robot_name}" filename="libgazebo_ros_p3d.so">
 		<bodyName>base_link</bodyName>
-		<frameName>odom</frameName>
+		<frameName>map</frameName>
 		<updateRate>10.0</updateRate>
-		<topicName>p3d_odom</topicName>
+		<topicName>${robot_name}/p3d_odom</topicName>
 		<xyzOffset>0 0 0</xyzOffset>
 		<rpyOffset>0 0 0</rpyOffset>

File: catkin_ws/src/duckiepond_vehicle/urdf/usv_gazebo_thrust_plugin.xacro (robot description, xacro)
@@ -1,8 +1,8 @@
 <?xml version="1.0"?>
 <robot xmlns:xacro="http://ros.org/wiki/xacro">
-  <xacro:macro name="usv_thrust_gazebo" params="name">
+  <xacro:macro name="usv_thrust_gazebo" params="name robot_name:=boat">
     <!--Gazebo Plugin for simulating WAM-V dynamics-->
     <gazebo >
-      <plugin name="usv_thrust_${name}" filename="libusv_gazebo_thrust_plugin.so">
+      <plugin name="usv_thrust_${robot_name}" filename="libusv_gazebo_thrust_plugin.so">
 	<bodyName>base_link</bodyName>
 	<!-- Which thruster curve to use -->
@@ -19,4 +19,5 @@
 	<maxForceRev>-100.0</maxForceRev>
 	<cmdTimeout>1.0</cmdTimeout>
+	<topicName>${robot_name}/cmd_drive</topicName>
       </plugin>
       </gazebo>

Commit message: update readme

File: catkin_ws/src/duckiepond_vehicle/urdf/duckieboat.xacro (robot description, xacro)
@@ -6,5 +6,5 @@
     <xacro:include filename="$(find duckiepond_vehicle)/urdf/usv_gazebo_imu_plugin.xacro" />
     <xacro:usv_imu name="imu" robot_name="$(arg robot_name)">
-        <origin xyz="0.2 0.0 0.5" rpy="0 0 0" />
+        <origin xyz="0.5 0.0 0.5" rpy="0 0 0" />
     </xacro:usv_imu>
     <!-- Attach p3d odometry plugin -->
@@ -14,5 +14,5 @@
     <xacro:include filename="$(find duckiepond_vehicle)/urdf/usv_gazebo_gps_plugin.xacro" />
     <xacro:usv_gps name="gps" latitude="24.788808" longitude="121.000188" altitude="2.5" robot_name="$(arg robot_name)">
-        <origin xyz="0.2 0.0 0.8" rpy="0 0 0" />
+        <origin xyz="0.5 0.0 0.8" rpy="0 0 0" />
     </xacro:usv_gps>
     <!-- Attach hydrodynamics plugin -->

File: catkin_ws/src/duckiepond_vehicle/urdf/usv_gazebo_gps_plugin.xacro (robot description, xacro)
@@ -5,5 +5,5 @@
       <visual>
         <geometry>
-          <box size="0.2 0.5 0.2" />
+          <box size="0.1 0.3 0.1" />
         </geometry>
       </visual>

Commit message: add two apriltag to duckiepond

File: catkin_ws/src/duckiepond_vehicle/urdf/duckieboat.xacro (robot description, xacro)
@@ -27,5 +27,5 @@
     <!-- Attach apriltag -->
     <xacro:include filename="$(find duckiepond_vehicle)/urdf/usv_gazebo_apriltags_plugin.xacro" />
-    <xacro:usv_apriltags name="top_tag" tag_id="$(arg robot_id)" tag_size="1.00">
+    <xacro:usv_apriltags name="top_tag" tag_id="$(arg robot_id)" tag2_id="$(arg robot_id2)" tag_size="1.00">
         <origin xyz="0.5 0 1" rpy="0 1.57 0"/>
     </xacro:usv_apriltags>

File: catkin_ws/src/duckiepond_vehicle/urdf/usv_gazebo_apriltags_plugin.xacro (robot description, xacro)
@@ -1,10 +1,20 @@
 <?xml version="1.0"?>
 <robot xmlns:xacro="http://ros.org/wiki/xacro">
-  <xacro:macro name="usv_apriltags" params="*origin name tag_id:=0 tag_size:=0.54">
+  <xacro:macro name="usv_apriltags" params="*origin name tag_id:=0 tag2_id:=1 tag_size:=0.54">
   <!--xacro:arg name="tag_id" default="0"/-->
     <link name="tag_link">
         <visual>
             <origin
-                xyz="0 0 0"
+                xyz="0 0 0.5"
+                rpy="0 0 0" />
+            <geometry>
+                <box size="0.01 ${tag_size} ${tag_size}"/>
+            </geometry>
+        </visual>
+    </link>
+    <link name="tag2_link">
+        <visual>
+            <origin
+                xyz="0 0 -0.5"
                 rpy="0 0 0" />
             <geometry>
@@ -18,8 +28,17 @@
       <child link="tag_link"/>
     </joint>
+    <joint name="tag2_joint" type="fixed">
+      <xacro:insert_block name="origin"/>
+      <parent link="base_link"/>
+      <child link="tag2_link"/>
+    </joint>
     <gazebo reference="tag_link">
         <turnGravityOff>true</turnGravityOff>
         <material>a_${tag_id}/Image</material>
     </gazebo>
+    <gazebo reference="tag2_link">
+        <turnGravityOff>true</turnGravityOff>
+        <material>a_${tag2_id}/Image</material>
+    </gazebo>
   </xacro:macro>
 </robot>

File: catkin_ws/src/duckiepond_vehicle/urdf/watchtower.xacro (robot description, xacro)
@@ -3,17 +3,7 @@
     <!-- Defines the base vehicle -->
     <xacro:include filename="$(find duckiepond_vehicle)/urdf/duckieboat_base.xacro"/>
-    <!-- Attach IMU plugin -->
-    <xacro:include filename="$(find duckiepond_vehicle)/urdf/usv_gazebo_imu_plugin.xacro" />
-    <xacro:usv_imu name="imu" robot_name="$(arg robot_name)">
-        <origin xyz="0.5 0.0 0.5" rpy="0 0 0" />
-    </xacro:usv_imu>
     <!-- Attach p3d odometry plugin -->
     <xacro:include filename="$(find duckiepond_vehicle)/urdf/usv_gazebo_p3d_plugin.xacro" />
     <xacro:usv_p3d name="p3d" robot_name="$(arg robot_name)"/>
-    <!-- Attach GPS plugin -->
-    <xacro:include filename="$(find duckiepond_vehicle)/urdf/usv_gazebo_gps_plugin.xacro" />
-    <xacro:usv_gps name="gps" latitude="24.788808" longitude="121.000188" altitude="2.5" robot_name="$(arg robot_name)">
-        <origin xyz="0.5 0.0 0.8" rpy="0 0 0" />
-    </xacro:usv_gps>
     <!-- Attach hydrodynamics plugin -->
     <xacro:include filename="$(find duckiepond_vehicle)/urdf/usv_gazebo_dynamics_plugin.xacro"/>

Commit message: fix camera error

File: catkin_ws/src/duckiepond_vehicle/urdf/duckieboat.xacro (robot description, xacro)
@@ -26,7 +26,7 @@
     <xacro:usv_camera name="camera" robot_name="$(arg robot_name)"/>
     <!-- Attach apriltag -->
-    <xacro:include filename="$(find duckiepond_vehicle)/urdf/usv_gazebo_apriltags_plugin.xacro" />
+    <!--xacro:include filename="$(find duckiepond_vehicle)/urdf/usv_gazebo_apriltags_plugin.xacro" />
     <xacro:usv_apriltags name="top_tag" tag_id="$(arg robot_id)" tag2_id="$(arg robot_id2)" tag_size="1.00">
         <origin xyz="0.5 0 1" rpy="0 1.57 0"/>
-    </xacro:usv_apriltags>
+    </xacro:usv_apriltags-->
 </robot>

File: catkin_ws/src/duckiepond_vehicle/urdf/usv_gazebo_camera_plugin.xacro (robot description, xacro)
@@ -4,10 +4,10 @@
   <!-- camera position -->
   <xacro:property name="origin_mid">
-    <origin xyz="0.52 0 ${camera_z}" rpy="0 ${camera_pitch} 0" />
+    <origin xyz="1.0 0 ${camera_z}" rpy="0 ${camera_pitch} 0" />
   </xacro:property>
   <!-- mid camera -->
   <link name="camera_link">
     <!--visual>
-      <origin xyz="-0.01 0 0" rpy="0 ${camera_pitch} 1.57"/>
+      <origin xyz="-0.01 0 0" rpy="0 ${camera_pitch} 0"/>
       <geometry>
         <mesh filename="model://zed/zed_model.dae" scale="0.02 0.02 0.02"/>
