Commit message: add watchtower, apriltag_base, duckiepond_apriltag

File: catkin_ws/src/duckiepond_vehicle/urdf/usv_gazebo_camera_plugin.xacro (robot description, xacro)
@@ -1,13 +1,13 @@
 <?xml version="1.0"?>
 <robot xmlns:xacro="http://ros.org/wiki/xacro">
-  <xacro:macro name="usv_camera" params="name robot_name:=duckieboat">
+  <xacro:macro name="usv_camera" params="name robot_name:=duckieboat camera_z:=0.45 camera_row:=1.57">
   <!-- camera position -->
   <xacro:property name="origin_mid">
-    <origin xyz="1 0 0.45" rpy="0 0 0" />
+    <origin xyz="1 0 ${camera_z}" rpy="0 0 0" />
   </xacro:property>
   <!-- mid camera -->
   <link name="camera_link">
     <visual>
-      <origin xyz="-0.01 0 0" rpy="1.57 0 1.57"/>
+      <origin xyz="-0.01 0 0" rpy="${camera_row} 0 1.57"/>
       <geometry>
         <mesh filename="model://zed/zed_model.dae" scale="0.02 0.02 0.02"/>

File: catkin_ws/src/duckiepond_vehicle/urdf/watchtower.xacro (robot description, xacro)
@@ -24,9 +24,4 @@
     <!-- Attach camera plugin -->
     <xacro:include filename="$(find duckiepond_vehicle)/urdf/usv_gazebo_camera_plugin.xacro"/>
-    <xacro:usv_camera name="camera" robot_name="$(arg robot_name)"/>
-    <!-- Attach apriltag -->
-    <xacro:include filename="$(find duckiepond_vehicle)/urdf/usv_gazebo_apriltags_plugin.xacro" />
-    <xacro:usv_apriltags name="top_tag" tag_id="512" tag_size="1.00">
-        <origin xyz="0.5 0 1" rpy="0 1.57 0"/>
-    </xacro:usv_apriltags>
+    <xacro:usv_camera name="camera" robot_name="$(arg robot_name)" camera_z="$(arg camera_z)" camera_row="$(arg camera_row)"/>
 </robot>

Commit message: upload new duckieboat model.  duckiepond_gazebo duckiepond_new.launch

File: catkin_ws/src/duckiepond_vehicle/urdf/usv_gazebo_camera_plugin.xacro (robot description, xacro)
@@ -1,17 +1,17 @@
 <?xml version="1.0"?>
 <robot xmlns:xacro="http://ros.org/wiki/xacro">
-  <xacro:macro name="usv_camera" params="name robot_name:=duckieboat camera_z:=0.45 camera_pitch:=0">
+  <xacro:macro name="usv_camera" params="name robot_name:=duckieboat camera_z:=0.44 camera_pitch:=0">
   <!-- camera position -->
   <xacro:property name="origin_mid">
-    <origin xyz="1 0 ${camera_z}" rpy="0 ${camera_pitch} 0" />
+    <origin xyz="0.52 0 ${camera_z}" rpy="0 ${camera_pitch} 0" />
   </xacro:property>
   <!-- mid camera -->
   <link name="camera_link">
-    <visual>
+    <!--visual>
       <origin xyz="-0.01 0 0" rpy="0 ${camera_pitch} 1.57"/>
       <geometry>
         <mesh filename="model://zed/zed_model.dae" scale="0.02 0.02 0.02"/>
       </geometry>
-    </visual>
+    </visual-->
   </link>
   <joint name="camera_joint" type="fixed">

File: catkin_ws/src/duckiepond_vehicle/urdf/usv_gazebo_dynamics_plugin.xacro (robot description, xacro)
@@ -7,5 +7,5 @@
 	<bodyName>base_link</bodyName>
 	<waterLevel>0</waterLevel> <!-- Must be same as the ocean model!-->
-	<waterDensity>997.8</waterDensity>
+	<waterDensity>443.22</waterDensity>
 	<cmdTimeout>1.0</cmdTimeout>
 	<!-- Added mass -->
@@ -21,5 +21,5 @@
 	<kP>50.0</kP>
 	<mQ>50.0</mQ>
-	<nR>800.0</nR>
+	<nR>400.0</nR>
 	<nRR>0.0</nRR>
 	<!-- General dimensions -->

File: catkin_ws/src/duckiepond_vehicle/urdf/usv_gazebo_gps_plugin.xacro (robot description, xacro)
@@ -3,9 +3,9 @@
   <xacro:macro name="usv_gps" params="*origin name longitude:=-157.8901 latitude:=21.30996 altitude:=1.5 robot_name:=boat">
     <link name="${name}">
-      <visual>
+      <!--visual>
         <geometry>
-          <box size="0.1 0.3 0.1" />
+          <box size="0.01 0.03 0.01" />
         </geometry>
-      </visual>
+      </visual-->
     </link>
     <joint name="${name}_joint" type="fixed">

File: catkin_ws/src/duckiepond_vehicle/urdf/usv_gazebo_imu_plugin.xacro (robot description, xacro)
@@ -3,9 +3,9 @@
   <xacro:macro name="usv_imu" params="*origin name robot_name:=boat">
     <link name="${name}">
-      <visual>
+      <!--visual>
         <geometry>
-          <box size="0.1 0.1 0.1" />
+          <box size="0.01 0.01 0.01" />
         </geometry>
-      </visual>
+      </visual-->
     </link>
     <joint name="${name}_joint" type="fixed">

Commit message: update launch fil

File: catkin_ws/src/duckiepond_vehicle/urdf/usv_gazebo_camera_plugin.xacro (robot description, xacro)
@@ -4,5 +4,5 @@
   <!-- camera position -->
   <xacro:property name="origin_mid">
-    <origin xyz="1.0 0 ${camera_z}" rpy="0 ${camera_pitch} 0" />
+    <origin xyz="0.52 0 ${camera_z}" rpy="0 ${camera_pitch} 0" />
   </xacro:property>
   <!-- mid camera -->
